Commit message: v1.0

File: RLEnv/BipedWalkerEnv/URDFs/biped.urdf (robot description, URDF)
Before this commit: robot biped, 7 links, 6 joints
Links:
- link torso: mass 40 -> 10

Commit message: v1.1

File: RLEnv/BipedWalkerEnv/URDFs/biped.urdf (robot description, URDF)
Before this commit: robot biped, 7 links, 6 joints
Links:
- link left_foot: geometry collision box size=0.2 0.2 0.1; visual box size=0.2 0.2 0.1
- link right_foot: geometry collision box size=0.2 0.2 0.1; visual box size=0.2 0.2 0.1
